Commit message: update s500 and s500_uam file with dae model rather than STL model

File: robots/s500_description/urdf/s500.urdf (robot description, URDF)
Before this commit: robot s500_quadrotor, 5 links, 4 joints
Joints:
- joint rotor_joint_1: origin xyz=0.171 0.171 0.045 rpy=0 0 0 -> xyz=0.171 0.171 0.07 rpy=0 0 0
- joint rotor_joint_2: origin xyz=-0.171 0.171 0.045 rpy=0 0 0 -> xyz=-0.171 0.171 0.07 rpy=0 0 0
- joint rotor_joint_3: origin xyz=-0.171 -0.171 0.045 rpy=0 0 0 -> xyz=-0.171 -0.171 0.07 rpy=0 0 0
- joint rotor_joint_4: origin xyz=0.1701 -0.1701 0.0603 rpy=0 0 0 -> xyz=0.1701 -0.1701 0.07 rpy=0 0 0

File: robots/s500_description/urdf/s500_uam.urdf (robot description, URDF)
Before this commit: robot s500_uam, 9 links, 8 joints
Links:
- link link_1: geometry collision mesh filename=package://example-robot-data/robots/s500_description/meshes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; visual mesh filename=package://example-robot-data/robots/s500_description/meshes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
- link link_2: geometry collision mesh filename=package://example-robot-data/robots/s500_description/meshes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; visual mesh filename=package://example-robot-data/robots/s500_description/meshes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
- link link_3: geometry collision mesh filename=package://example-robot-data/robots/s500_description/meshes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; visual mesh filename=package://example-robot-data/robots/s500_description/meshes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
- link link_4: geometry collision mesh filename=package://example-robot-data/robots/s500_description/meshes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; visual mesh filename=package://example-robot-data/robots/s500_description/meshes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
Joints:
- joint joint_1: axis 0 0 1 -> 0 1 0
- joint joint_2: axis 0 0 1 -> 0 1 0; origin xyz=0 0 -0.09925 rpy=0 0.2936 0 -> xyz=0 0 -0.09925 rpy=0 0 0
- joint rotor_joint_1: origin xyz=0.171 0.171 0.045 rpy=0 0 0 -> xyz=0.171 0.171 0.07 rpy=0 0 0
- joint rotor_joint_2: origin xyz=-0.171 0.171 0.045 rpy=0 0 0 -> xyz=-0.171 0.171 0.07 rpy=0 0 0
- joint rotor_joint_3: origin xyz=-0.171 -0.171 0.045 rpy=0 0 0 -> xyz=-0.171 -0.171 0.07 rpy=0 0 0
- joint rotor_joint_4: origin xyz=0.1701 -0.1701 0.0603 rpy=0 0 0 -> xyz=0.1701 -0.1701 0.07 rpy=0 0 0
