Commit message: change the default joint position for s500_uam

File: robots/s500_description/urdf/s500_uam.urdf (robot description, URDF)
Before this commit: robot s500_uam, 9 links, 8 joints
Joints:
- joint joint_1: origin xyz=0.0007 0 -0.07275 rpy=0 0 0 -> xyz=0.0007 0 -0.07275 rpy=0 -1 0
- joint joint_2: origin xyz=0 0 -0.09925 rpy=0 0 0 -> xyz=0 0 -0.09925 rpy=0 -0.6 0
