Commit message: update s500 uam urdf file, add gripper link and fixed the rotor joint angle

File: robots/s500_description/s500_uam/urdf/s500_uam.urdf (robot description, URDF)
Before this commit: robot s500_uam, 9 links, 8 joints
Links:
- added link gripper_link; visual box size=0.01 0.01 0.01
- link base_link: geometry collision mesh filename=package://example-robot-data/robots/s500_description/s500_u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; visual mesh filename=package://example-robot-data/robots/s500_description/s500_u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
- link link_1: geometry collision mesh filename=package://example-robot-data/robots/s500_description/s500_u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; visual mesh filename=package://example-robot-data/robots/s500_description/s500_u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
- link link_2: geometry collision mesh filename=package://example-robot-data/robots/s500_description/s500_u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; visual mesh filename=package://example-robot-data/robots/s500_description/s500_u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
- link link_3: geometry collision mesh filename=package://example-robot-data/robots/s500_description/s500_u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; visual mesh filename=package://example-robot-data/robots/s500_description/s500_u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
- link link_4: geometry collision mesh filename=package://example-robot-data/robots/s500_description/s500_u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; visual mesh filename=package://example-robot-data/robots/s500_description/s500_u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
- link rotor_1: geometry collision mesh filename=package://example-robot-data/robots/s500_description/s500_u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; visual mesh filename=package://example-robot-data/robots/s500_description/s500_u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
- link rotor_2: geometry collision mesh filename=package://example-robot-data/robots/s500_description/s500_u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; visual mesh filename=package://example-robot-data/robots/s500_description/s500_u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
- link rotor_3: geometry collision mesh filename=package://example-robot-data/robots/s500_description/s500_u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; visual mesh filename=package://example-robot-data/robots/s500_description/s500_u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
- link rotor_4: geometry collision mesh filename=package://example-robot-data/robots/s500_description/s500_u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; visual mesh filename=package://example-robot-data/robots/s500_description/s500_u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
Joints:
- added joint gripper_joint: type fixed, parent link_2, child gripper_link, origin xyz=0 0 -0.14 rpy=0 0 0
- joint joint_1: limit (none) -> lower=-1.5 upper=1.5 effort=1 velocity=3; origin xyz=0.0007 0 -0.07275 rpy=0 -1 0 -> xyz=0.0007 0 -0.07275 rpy=0 0 0; type continuous -> revolute
- joint joint_2: limit (none) -> lower=-1.5 upper=1.5 effort=1 velocity=3; origin xyz=0 0 -0.09925 rpy=0 -0.6 0 -> xyz=0 0 -0.09925 rpy=0 0 0; type continuous -> revolute
- joint rotor_joint_1: axis 0 1 0 -> 0 0 1; origin xyz=0.171 0.171 0.045 rpy=0 0 0 -> xyz=0.171 0.171 0.07 rpy=0 0 0
- joint rotor_joint_2: axis 0 1 0 -> 0 0 1; origin xyz=-0.171 0.171 0.045 rpy=0 0 0 -> xyz=-0.171 0.171 0.07 rpy=0 0 0
- joint rotor_joint_3: axis 0 1 0 -> 0 0 1; origin xyz=-0.171 -0.171 0.045 rpy=0 0 0 -> xyz=-0.171 -0.171 0.07 rpy=0 0 0
- joint rotor_joint_4: axis 0 1 0 -> 0 0 1; origin xyz=0.1701 -0.1701 0.0603 rpy=0 0 0 -> xyz=0.1701 -0.1701 0.07 rpy=0 0 0

File: robots/s500_description/s500_uam/urdf/s500_uam_simple.urdf (robot description, URDF)
Before this commit: robot s500_uam, 9 links, 8 joints
Links:
- added link gripper_link; visual box size=0.01 0.01 0.01
- link base_link: geometry collision mesh filename=package://example-robot-data/robots/s500_description/s500_u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; visual mesh filename=package://example-robot-data/robots/s500_description/s500_u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
- link link_1: geometry collision mesh filename=package://example-robot-data/robots/s500_description/s500_u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; visual mesh filename=package://example-robot-data/robots/s500_description/s500_u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
- link link_2: geometry collision mesh filename=package://example-robot-data/robots/s500_description/s500_u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; visual mesh filename=package://example-robot-data/robots/s500_description/s500_u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
- link link_3: geometry collision mesh filename=package://example-robot-data/robots/s500_description/s500_u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; visual mesh filename=package://example-robot-data/robots/s500_description/s500_u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
- link link_4: geometry collision mesh filename=package://example-robot-data/robots/s500_description/s500_u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; visual mesh filename=package://example-robot-data/robots/s500_description/s500_u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
- link rotor_1: geometry collision mesh filename=package://example-robot-data/robots/s500_description/s500_u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; visual mesh filename=package://example-robot-data/robots/s500_description/s500_u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
- link rotor_2: geometry collision mesh filename=package://example-robot-data/robots/s500_description/s500_u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; visual mesh filename=package://example-robot-data/robots/s500_description/s500_u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
- link rotor_3: geometry collision mesh filename=package://example-robot-data/robots/s500_description/s500_u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; visual mesh filename=package://example-robot-data/robots/s500_description/s500_u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
- link rotor_4: geometry collision mesh filename=package://example-robot-data/robots/s500_description/s500_u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; visual mesh filename=package://example-robot-data/robots/s500_description/s500_u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
Joints:
- added joint gripper_joint: type fixed, parent link_2, child gripper_link, origin xyz=0 0 -0.14 rpy=0 0 0
- joint joint_1: origin xyz=0.0007 0 -0.07275 rpy=0 -1 0 -> xyz=0.0007 0 -0.07275 rpy=0 0 0
- joint joint_2: origin xyz=0 0 -0.09925 rpy=0 -0.6 0 -> xyz=0 0 -0.09925 rpy=0 0 0
