Commit message: update s500_uam_simple.urdf file

File: robots/s500_description/s500_uam/urdf/s500_uam_simple.urdf (robot description, URDF)
Before this commit: robot s500_uam, 10 links, 9 joints
Joints:
- joint joint_3: limit (none) -> lower=-1.57 upper=0 effort=10 velocity=1
- joint joint_4: limit (none) -> lower=0 upper=1.57 effort=10 velocity=1
